File: HAT with LowPass filters/HAT with LowPass filters.kicad_pcb (KiCad board)
At the start: 2 copper layers, 65 x 56.2 mm, 88 parts, among them IC1 SX1255, J1 U.FL, J2 U.FL, J3 RPi, J4 WP, Q1 BSS84, U1 MCP1703Ax-330xxDB, U2 24LC256, U3 74LVC1G74DP_125, U4 TQP3M9036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

Commit message: Add files via upload
Parts:
- moved REF** 5.25 mm to (137.2, 118.8)
Routing:
- net GND: track 14.5 -> 17.0 mm
- net /H_GPIO12: track 25.8 -> 26.0 mm, vias 2 -> 1
Other:
- board text removed: "V1.3.2"
Changed lines of the file:
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@@
 	(title_block
 		(title "SX1255-SXceiver-HAT")
-		(date "2026-03-15")
-		(rev "V1.3.2 FINAL")
+		(date "2026-03-23")
+		(rev "V1.3.3 FINAL")
 		(company "Z32IT")
 		(comment 1 "Modified SXceiver")
@@
 	(footprint "Symbol:OSHW-Logo_5.7x6mm_SilkScreen"
 		(layer "F.Cu")
-		(at 132 118.75)
+		(at 137.25 118.75)
 		(descr "Open Source Hardware Logo")
 		(tags "Logo OSHW")
@@
 		)
 	)
-	(gr_text "V1.3.2"
-		(at 136.5 121.5 0)
-		(layer "F.SilkS")
-		(effects
-			(font
-				(size 1 1)
-				(thickness 0.25)
-				(bold yes)
-			)
-			(justify left bottom)
-		)
-	)
 	(gr_text "GPIO13"
 		(at 158.75 96.75 90)
@@
 	)
 	(gr_text "HAT with LPF"
-		(at 118.25 121.5 0)
+		(at 122.75 121.75 0)
 		(layer "F.SilkS")
 		(effects
@@
 	)
 	(gr_text "Z32IT"
-		(at 120.25 119 0)
+		(at 124.75 119.25 0)
 		(layer "F.SilkS")
 		(effects
@@
 		(start 134.932 103.25)
 		(end 133.756 103.25)
-		(width 0.2)
+		(width 0.25)
 		(layer "F.Cu")
 		(net 2)
@@
 	)
 	(segment
+		(start 131.232 106.518)
+		(end 131 106.75)
+		(width 0.25)
+		(layer "F.Cu")
+		(net 2)
+	)
+	(segment
 		(start 133.756 103.25)
 		(end 133.244 103.762)
@@
 		(start 133.732 105.45)
 		(end 133.732 104.25)
-		(width 0.2)
+		(width 0.25)
 		(layer "F.Cu")
 		(net 2)
@@
 		(start 134.932 101.75)
 		(end 133.732 101.75)
-		(width 0.2)
+		(width 0.25)
 		(layer "F.Cu")
 		(net 2)
@@
 		(start 131.232 105.45)
 		(end 131.232 104.25)
-		(width 0.2)
+		(width 0.25)
 		(layer "F.Cu")
 		(net 2)
@@
 	)
 	(segment
+		(start 133.732 105.45)
+		(end 133.732 106.232)
+		(width 0.25)
+		(layer "F.Cu")
+		(net 2)
+	)
+	(segment
+		(start 131.232 105.45)
+		(end 131.232 106.518)
+		(width 0.25)
+		(layer "F.Cu")
+		(net 2)
+	)
+	(segment
+		(start 133.732 106.232)
+		(end 134 106.5)
+		(width 0.25)
+		(layer "F.Cu")
+		(net 2)
+	)
+	(segment
 		(start 142.505 114.105)
 		(end 142.5 114.11)
@@
 		(start 132.232 105.45)
 		(end 132.232 104.274)
-		(width 0.2)
+		(width 0.25)
 		(layer "F.Cu")
 		(net 2)
@@
 	)
 	(segment
-		(start 146.73 72.23)
-		(end 147.5 73)
-		(width 0.25)
-		(layer "F.Cu")
-		(net 45)
-	)
-	(segment
 		(start 146.47 72.23)
 		(end 146.73 72.23)
@@
 		(net 45)
 	)
-	(via
-		(at 147.5 73)
-		(size 0.6)
-		(drill 0.3)
-		(layers "F.Cu" "B.Cu")
-		(net 45)
-	)
 	(segment
-		(start 159.25 84.75)
-		(end 160 85.5)
+		(start 157.5 73.5)
+		(end 147.74 73.5)
 		(width 0.25)
 		(layer "B.Cu")
@@
 	)
 	(segment
-		(start 159.25 76.5)
-		(end 159.25 84.75)
+		(start 158.5 74.5)
+		(end 157.5 73.5)
 		(width 0.25)
 		(layer "B.Cu")
@@
 	)
 	(segment
-		(start 147.5 73)
-		(end 148 73.5)
+		(start 160 85.5)
+		(end 159.25 84.75)
 		(width 0.25)
 		(layer "B.Cu")
@@
 	)
 	(segment
-		(start 158.5 75.75)
-		(end 159.25 76.5)
+		(start 159.25 76.5)
+		(end 158.5 75.75)
 		(width 0.25)
 		(layer "B.Cu")
@@
 	)
 	(segment
-		(start 157.5 73.5)
+		(start 158.5 75.75)
 		(end 158.5 74.5)
 		(width 0.25)
@@
 	)
 	(segment
-		(start 148 73.5)
-		(end 157.5 73.5)
+		(start 147.74 73.5)
+		(end 146.47 72.23)
 		(width 0.25)
 		(layer "B.Cu")
@@
 	)
 	(segment
-		(start 158.5 74.5)
-		(end 158.5 75.75)
+		(start 159.25 84.75)
+		(end 159.25 76.5)
 		(width 0.25)
 		(layer "B.Cu")
