File: HAT with BandPass filters/HAT with BandPass filters.kicad_pcb (KiCad board)
At the start: 2 copper layers, 65 x 56.2 mm, 88 parts, among them IC1 SX1255, J1 TX_SMA, J2 RX_SMA, J3 RPi, J4 WP, Q1 BSS84, U1 MCP1703Ax-330xxDB, U2 24LC256, U3 74LVC1G74DP_125, U4 TQP3M9036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

Commit message: Add files via upload
Parts:
- moved REF** 9.26 mm to (136.5, 119.5)
Routing:
- net GND: track 14.5 -> 16.9 mm
- net /H_GPIO12: vias 2 -> 1
Other:
- board text removed: "V1.4.3"
Changed lines of the file:
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@@
 	(title_block
 		(title "SX1255-SXceiver-HAT with BPF")
-		(date "2026-03-15")
-		(rev "V1.4.3 Final")
+		(date "2026-03-23")
+		(rev "V1.4.4 Final")
 		(company "Z32IT")
 		(comment 1 "Modified SXceiver")
@@
 	(footprint "Symbol:OSHW-Logo_5.7x6mm_SilkScreen"
 		(layer "F.Cu")
-		(at 127.25 120)
+		(at 136.5 119.5)
 		(descr "Open Source Hardware Logo")
 		(tags "Logo OSHW")
@@
 	)
 	(gr_text "HAT with BPF"
-		(at 112.5 121.75 0)
+		(at 119.75 122 0)
 		(layer "F.SilkS")
 		(effects
@@
 		)
 	)
-	(gr_text "V1.4.3"
-		(at 132.25 120.75 0)
-		(layer "F.SilkS")
-		(effects
-			(font
-				(size 1 1)
-				(thickness 0.25)
-				(bold yes)
-			)
-			(justify left bottom)
-		)
-	)
 	(gr_text "DIO0"
 		(at 104.25 99 0)
@@
 	)
 	(gr_text "Z32IT"
-		(at 115 119.75 0)
+		(at 122.25 120 0)
 		(layer "F.SilkS")
 		(effects
@@
 		(start 134.932 103.25)
 		(end 133.756 103.25)
-		(width 0.2)
+		(width 0.25)
 		(layer "F.Cu")
 		(net 2)
@@
 	)
 	(segment
+		(start 133.732 106.232)
+		(end 133.875 106.375)
+		(width 0.25)
+		(layer "F.Cu")
+		(net 2)
+	)
+	(segment
 		(start 140.255 113.25)
 		(end 140.255 114.355)
@@
 	)
 	(segment
+		(start 133.732 105.45)
+		(end 133.732 106.232)
+		(width 0.25)
+		(layer "F.Cu")
+		(net 2)
+	)
+	(segment
 		(start 140.255 113.25)
 		(end 140.255 112.75)
@@
 	)
 	(segment
+		(start 131.232 106.518)
+		(end 131 106.75)
+		(width 0.25)
+		(layer "F.Cu")
+		(net 2)
+	)
+	(segment
 		(start 133.756 103.25)
 		(end 133.244 103.762)
@@
 		(start 133.732 105.45)
 		(end 133.732 104.25)
-		(width 0.2)
+		(width 0.25)
 		(layer "F.Cu")
 		(net 2)
@@
 		(start 134.932 101.75)
 		(end 133.732 101.75)
-		(width 0.2)
+		(width 0.25)
 		(layer "F.Cu")
 		(net 2)
@@
 		(start 131.232 105.45)
 		(end 131.232 104.25)
-		(width 0.2)
+		(width 0.25)
 		(layer "F.Cu")
 		(net 2)
@@
 	)
 	(segment
+		(start 131.232 105.45)
+		(end 131.232 106.518)
+		(width 0.25)
+		(layer "F.Cu")
+		(net 2)
+	)
+	(segment
 		(start 132.232 105.45)
 		(end 132.232 104.274)
-		(width 0.2)
+		(width 0.25)
 		(layer "F.Cu")
 		(net 2)
@@
 	)
 	(segment
-		(start 146.48 72.23)
-		(end 147.5 73.25)
-		(width 0.2)
-		(layer "F.Cu")
-		(net 55)
-	)
-	(segment
 		(start 146.47 72.23)
 		(end 146.48 72.23)
@@
 	)
 	(via
-		(at 147.5 73.25)
-		(size 0.6)
-		(drill 0.3)
-		(layers "F.Cu" "B.Cu")
-		(net 55)
-	)
-	(via
 		(at 159.75 85.775)
 		(size 0.6)
@@
 	)
 	(segment
-		(start 147.5 73.25)
-		(end 147.75 73.5)
+		(start 159 75)
+		(end 157.5 73.5)
 		(width 0.2)
 		(layer "B.Cu")
@@
 	)
 	(segment
-		(start 157.5 73.5)
-		(end 159 75)
+		(start 159.75 85.775)
+		(end 159 85.025)
 		(width 0.2)
 		(layer "B.Cu")
@@
 	)
 	(segment
-		(start 159 75)
-		(end 159 85.025)
+		(start 157.5 73.5)
+		(end 147.74 73.5)
 		(width 0.2)
 		(layer "B.Cu")
@@
 	)
 	(segment
-		(start 147.75 73.5)
-		(end 157.5 73.5)
+		(start 159 85.025)
+		(end 159 75)
 		(width 0.2)
 		(layer "B.Cu")
@@
 	)
 	(segment
-		(start 159 85.025)
-		(end 159.75 85.775)
+		(start 147.74 73.5)
+		(end 146.47 72.23)
 		(width 0.2)
 		(layer "B.Cu")
