File: HAT_MicroSpot/HAT_MicroSpot.kicad_pcb (KiCad board)
At the start: 2 copper layers, 65 x 56.2 mm, 85 parts, among them IC1 SX1255, J3 RPi, J4 WP, Q1 BSS84, U1 MCP1703Ax-330xxDB, U2 24LC256, U3 74LVC1G74DP_125, X1 TA0655A, X2 TA1761A, Y1 38.4MHZ

Commit message: Add files via upload
Routing:
- net GND: track 9.47 -> 11.8 mm
- net /H_GPIO12: vias 2 -> 1
Changed lines of the file:
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@@
 	(title_block
 		(title "HAT MicroSpot")
-		(date "2026-03-16")
+		(date "2026-03-23")
 		(rev "V1.5 Final")
 		(company "Z32IT")
@@
 		(start 134.932 103.25)
 		(end 133.756 103.25)
-		(width 0.2)
+		(width 0.25)
 		(layer "F.Cu")
 		(net 2)
@@
 	)
 	(segment
+		(start 131.232 105.45)
+		(end 131.232 106.768)
+		(width 0.25)
+		(layer "F.Cu")
+		(net 2)
+	)
+	(segment
 		(start 133.732 105.45)
 		(end 133.732 104.25)
-		(width 0.2)
+		(width 0.25)
 		(layer "F.Cu")
 		(net 2)
@@
 		(start 134.932 101.75)
 		(end 133.732 101.75)
-		(width 0.2)
+		(width 0.25)
 		(layer "F.Cu")
 		(net 2)
@@
 		(start 131.232 105.45)
 		(end 131.232 104.25)
-		(width 0.2)
+		(width 0.25)
+		(layer "F.Cu")
+		(net 2)
+	)
+	(segment
+		(start 133.732 105.45)
+		(end 133.732 106.482)
+		(width 0.25)
 		(layer "F.Cu")
 		(net 2)
@@
 		(start 132.232 105.45)
 		(end 132.232 104.274)
-		(width 0.2)
+		(width 0.25)
 		(layer "F.Cu")
 		(net 2)
@@
 	)
 	(segment
-		(start 146.48 72.23)
-		(end 147.5 73.25)
-		(width 0.2)
-		(layer "F.Cu")
-		(net 53)
-	)
-	(segment
 		(start 146.47 72.23)
 		(end 146.48 72.23)
@@
 	)
 	(via
-		(at 147.5 73.25)
-		(size 0.6)
-		(drill 0.3)
-		(layers "F.Cu" "B.Cu")
-		(net 53)
-	)
-	(via
 		(at 159.75 85.775)
 		(size 0.6)
@@
 		(start 147.5 73.25)
 		(end 147.75 73.5)
-		(width 0.2)
+		(width 0.25)
 		(layer "B.Cu")
 		(net 53)
@@
 		(start 157.5 73.5)
 		(end 159 75)
-		(width 0.2)
+		(width 0.25)
 		(layer "B.Cu")
 		(net 53)
@@
 		(start 159 75)
 		(end 159 85.025)
-		(width 0.2)
+		(width 0.25)
 		(layer "B.Cu")
 		(net 53)
@@
 		(start 147.75 73.5)
 		(end 157.5 73.5)
-		(width 0.2)
+		(width 0.25)
 		(layer "B.Cu")
 		(net 53)
@@
 		(start 159 85.025)
 		(end 159.75 85.775)
+		(width 0.25)
+		(layer "B.Cu")
+		(net 53)
+	)
+	(segment
+		(start 147.5 73.25)
+		(end 147.49 73.25)
 		(width 0.2)
 		(layer "B.Cu")
@@
 	)
 	(segment
+		(start 147.49 73.25)
+		(end 146.47 72.23)
+		(width 0.25)
+		(layer "B.Cu")
+		(net 53)
+	)
+	(segment
 		(start 147.5 92.575)
 		(end 147.5 95)
@@
 		(start 150 75.76)
 		(end 150 76.75)
-		(width 0.2)
+		(width 0.25)
 		(layer "F.Cu")
 		(net 56)
@@
 		(start 149.01 74.77)
 		(end 150 75.76)
-		(width 0.2)
+		(width 0.25)
 		(layer "F.Cu")
 		(net 56)
@@
 		(start 158 76.75)
 		(end 158 85.775)
-		(width 0.2)
+		(width 0.25)
 		(layer "B.Cu")
 		(net 56)
@@
 		(start 150 76.75)
 		(end 158 76.75)
-		(width 0.2)
+		(width 0.25)
 		(layer "B.Cu")
 		(net 56)

Commit message: Add files via upload
Parts:
- E2: value TX-CHP -> RX-CHP
- X2: value TA1761A -> TA2490A; footprint Filter:Filter_SAW-8_3.8x3.8mm -> Filter:Filter_SAW_Epcos_DCC6C_3x3mm
- moved X2 0.58 mm to (147.3, 112.2)
Connections:
- R26 pad 1: Net-(X2-RF_out) -> Net-(X2-OUT)
- X2 pad 5: GND -> Net-(X2-OUT)
- X2 pad 6: Net-(X2-RF_out) -> GND
Routing:
- net Net-(X2-OUT): track 0.00 -> 9.56 mm
- net Net-(X2-RF_out): track 8.55 -> 0.00 mm
- net Net-(X2-IN): track 6.21 -> 5.61 mm
- net GND: vias 426 -> 429
