File: HAT_MicroSpot/HAT_MicroSpot.kicad_sch (KiCad schematic)
At the start: 84 parts, among them IC1 SX1255, J3 RPi, J4 WP, Q1 BSS84, U1 MCP1703Ax-330xxDB, U2 24LC256, U3 74LVC1G74DP_125, X1 TA0655A, X2 TA1761A, Y1 38.4MHZ

Commit message: Add files via upload
Parts:
- removed X2: TA1761A, Filter:Filter_SAW-8_3.8x3.8mm, symbol TA1761A_:TA1761A
- added X2: TA2490A, Filter:Filter_SAW_Epcos_DCC6C_3x3mm, symbol RF_Filter:B3715
Connections:
- net GND: now also X2.1 (GND), X2.3 (GND), X2.4 (GND), X2.6 (GND)
- net at R26.1: now also X2.5 (OUT)
- net at C19.2: now also X2.2 (IN)
Changed lines of the file:
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@@
 	(title_block
 		(title "HAT MicroSpot")
-		(date "2026-03-16")
-		(rev "V1.5  Final")
+		(date "2026-03-30")
+		(rev "V1.6")
 		(company "Z32IT")
 		(comment 1 "Modified SXceiver")
@@
 	(wire
 		(pts
+			(xy 184.15 43.18) (xy 184.15 50.8)
+		)
+		(stroke
+			(width 0)
+			(type default)
+		)
+	)
+	(wire
+		(pts
 			(xy 276.86 218.44) (xy 280.67 218.44)
 		)
@@
 	(wire
 		(pts
+			(xy 189.23 60.96) (xy 200.66 60.96)
+		)
+		(stroke
+			(width 0)
+			(type default)
+		)
+	)
+	(wire
+		(pts
 			(xy 59.69 110.49) (xy 57.15 110.49)
 		)
@@
 	(wire
 		(pts
-			(xy 158.75 60.96) (xy 165.1 60.96)
+			(xy 157.48 93.98) (xy 161.29 93.98)
 		)
 		(stroke
@@
 	(wire
 		(pts
-			(xy 157.48 93.98) (xy 161.29 93.98)
+			(xy 218.44 85.09) (xy 218.44 86.36)
 		)
 		(stroke
@@
 	(wire
 		(pts
-			(xy 218.44 85.09) (xy 218.44 86.36)
+			(xy 52.07 177.8) (xy 52.07 179.07)
 		)
 		(stroke
@@
 	(wire
 		(pts
-			(xy 52.07 177.8) (xy 52.07 179.07)
+			(xy 355.6 146.05) (xy 358.14 146.05)
 		)
 		(stroke
@@
 	(wire
 		(pts
-			(xy 355.6 146.05) (xy 358.14 146.05)
+			(xy 158.75 60.96) (xy 168.91 60.96)
 		)
 		(stroke
@@
 	(wire
 		(pts
-			(xy 185.42 66.04) (xy 185.42 68.58)
-		)
-		(stroke
-			(width 0)
-			(type default)
-		)
-	)
-	(wire
-		(pts
 			(xy 179.07 93.98) (xy 187.96 93.98)
 		)
@@
 	(wire
 		(pts
-			(xy 185.42 60.96) (xy 200.66 60.96)
-		)
-		(stroke
-			(width 0)
-			(type default)
-		)
-	)
-	(wire
-		(pts
 			(xy 358.14 130.81) (xy 355.6 130.81)
 		)
@@
 	)
 	(symbol
+		(lib_id "RF_Filter:B3715")
+		(at 179.07 60.96 180)
+		(unit 1)
+		(exclude_from_sim no)
+		(in_bom yes)
+		(on_board yes)
+		(dnp no)
+		(fields_autoplaced yes)
+		(property "Reference" "X2"
+			(at 179.07 69.85 0)
+			(effects
+				(font
+					(size 1.27 1.27)
+				)
+			)
+		)
+		(property "Value" "TA2490A"
+			(at 179.07 72.39 0)
+			(effects
+				(font
+					(size 1.27 1.27)
+				)
+			)
+		)
+		(property "Footprint" "Filter:Filter_SAW_Epcos_DCC6C_3x3mm"
+			(at 179.07 60.96 0)
+			(effects
+				(font
+					(size 1.27 1.27)
+				)
+				(hide yes)
+			)
+		)
+		(property "Datasheet" ""
+			(at 179.07 60.96 0)
+			(effects
+				(font
+					(size 1.27 1.27)
+				)
+				(hide yes)
+			)
+		)
+		(property "Description" ""
+			(at 179.07 60.96 0)
+			(effects
+				(font
+					(size 1.27 1.27)
+				)
+				(hide yes)
+			)
+		)
+		(pin "4"
+		)
+		(pin "1"
+		)
+		(pin "5"
+		)
+		(pin "6"
+		)
+		(pin "3"
+		)
+		(pin "2"
+		)
+		(instances
+			(project ""
+				(path "/5946dd4e-fab1-4214-b6c7-4fabd0e98d1f"
+					(reference "X2")
+					(unit 1)
+				)
+			)
+		)
+	)
+	(symbol
 		(lib_id "Device:C_Small")
 		(at 220.98 215.9 270)
@@
 	)
 	(symbol
-		(lib_id "TA1761A_:TA1761A")
-		(at 175.26 63.5 180)
-		(unit 1)
-		(exclude_from_sim no)
-		(in_bom yes)
-		(on_board yes)
-		(dnp no)
-		(fields_autoplaced yes)
-		(property "Reference" "X2"
-			(at 175.26 49.53 0)
-			(effects
-				(font
-					(size 1.27 1.27)
-				)
-			)
-		)
-		(property "Value" "TA1761A"
-			(at 175.26 52.07 0)
-			(effects
-				(font
-					(size 1.27 1.27)
-				)
-			)
-		)
-		(property "Footprint" "Filter:Filter_SAW-8_3.8x3.8mm"
-			(at 175.26 54.61 0)
-			(effects
-				(font
-					(size 1.27 1.27)
-				)
-			)
-		)
-		(property "Datasheet" ""
-			(at 180.34 72.39 0)
-			(effects
-				(font
-					(size 1.27 1.27)
-				)
-				(hide yes)
-			)
-		)
-		(property "Description" "Bandpass Filter, 440MHz, BW-1MHz, SAW filter 8-pin"
-			(at 175.26 63.5 0)
-			(effects
-				(font
-					(size 1.27 1.27)
-				)
-				(hide yes)
-			)
-		)
-		(pin "4"
-		)
-		(pin "8"
-		)
-		(pin "7"
-		)
-		(pin "2"
-		)
-		(pin "3"
-		)
-		(pin "6"
-		)
-		(pin "1"
-		)
-		(pin "5"
-		)
-		(instances
-			(project "SX1255-SXCEIVER-HAT with BPF"
-				(path "/5946dd4e-fab1-4214-b6c7-4fabd0e98d1f"
-					(reference "X2")
-					(unit 1)
-				)
-			)
-		)
-	)
-	(symbol
 		(lib_id "power:GND")
 		(at 365.76 199.39 0)
@@
 	(symbol
 		(lib_id "power:GND")
-		(at 185.42 68.58 0)
+		(at 184.15 43.18 180)
 		(unit 1)
 		(exclude_from_sim no)
@@
 		(fields_autoplaced yes)
 		(property "Reference" "#PWR044"
-			(at 185.42 74.93 0)
+			(at 184.15 36.83 0)
 			(effects
 				(font
@@
 		)
 		(property "Value" "GND"
-			(at 187.96 69.8499 0)
+			(at 186.69 41.9099 0)
 			(effects
 				(font
 					(size 1.27 1.27)
 				)
-				(justify left)
+				(justify right)
 			)
 		)
 		(property "Footprint" ""
-			(at 185.42 68.58 0)
+			(at 184.15 43.18 0)
 			(effects
 				(font
@@
 		)
 		(property "Datasheet" ""
-			(at 185.42 68.58 0)
+			(at 184.15 43.18 0)
 			(effects
 				(font
@@
 		)
 		(property "Description" ""
-			(at 185.42 68.58 0)
+			(at 184.15 43.18 0)
 			(effects
 				(font
