File: HAT with PA/HAT with PA.kicad_pcb (KiCad board)
At the start: 2 copper layers, 65 x 56.2 mm, 89 parts, among them IC1 SX1255, J1 U.FL, J2 U.FL, J3 RPi, J4 WP, Q1 BSS84, U1 MCP1703Ax-330xxDB, U2 24LC256, U3 74LVC1G74DP_125, U4 TQP3M9036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

Commit message: Add files via upload
Parts:
- removed the REF** at (152.5, 119.8)
- added REF**: OSHW-Logo2_7.3x6mm_Copper, Symbol:OSHW-Logo2_7.3x6mm_Copper, F.Cu at (153.8, 122.2)
- D1: value White -> Red
- D6: value Green -> Yellow
- D7: value Green -> White
Other:
- board text added: "Little PA"
- board text removed: "HAT with L/BPF"
