File: HAT with PA/HAT with PA.kicad_sch (KiCad schematic)
At the start: 88 parts, among them IC1 SX1255, J1 U.FL, J2 U.FL, J3 RPi, J4 WP, Q1 BSS84, U1 MCP1703Ax-330xxDB, U2 24LC256, U3 74LVC1G74DP_125, U4 TQP3M9036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

Commit message: Add files via upload
Parts:
- D1: value White -> Red; Manufacturer Product Number LTST-T180UWET -> LTST-S270KRKT; Part Number 160-LTST-T180UWETCT-ND -> 160-1479-1-ND
- D2, D3, R34, R35: now in the parts list
- D6: value Green -> Yellow; Manufacturer Kingbright -> Lite-On Inc.; Manufacturer Product Number APT1608SGD3 -> LTST-C190KSKT; Part Number 754-APT1608SGD3CT-ND -> 160-1437-1-ND
- D7: value Green -> White; Manufacturer Kingbright -> Lite-On Inc.; Manufacturer Product Number APT1608SGD3 -> LTST-T180UWET; Part Number 754-APT1608SGD3CT-ND -> 160-LTST-T180UWETCT-ND
- U5: DigiKey Part Number (none) -> SRV05-4CT-ND; Manufacturer (none) -> Semtech Corporation; Manufacturer Product Number (none) -> SRV05-4.TCT; now left out of the parts list
- X1: Aliexpress (none) -> https://www.aliexpress.com/item/1005010661905531.html?spm=a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; now left out of the parts list
Other:
- title: HAT with LPF & BPF filters and SPI line protection -> HAT little PA
Changed lines of the file:
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@@
 	(paper "A3")
 	(title_block
-		(title "HAT with LPF & BPF filters and SPI line protection")
-		(date "2026-03-30")
-		(rev "V1.2")
+		(title "HAT little PA")
+		(date "2026-04-08")
+		(rev "V1.3")
 		(company "Z32IT")
 		(comment 1 "Modified SXceiver")
@@
 		(unit 1)
 		(exclude_from_sim no)
-		(in_bom yes)
+		(in_bom no)
 		(on_board yes)
 		(dnp no)
@@
 			)
 		)
+		(property "Aliexpress" "https://www.aliexpress.com/item/1005010661905531.html?spm=a2g0o.order_detail.order_detail_item.4.56ebf19cmfwY3c"
+			(at 273.05 68.58 0)
+			(effects
+				(font
+					(size 1.27 1.27)
+				)
+				(hide yes)
+			)
+		)
 		(pin "4"
 		)
@@
 		(at 351.79 195.58 270)
 		(unit 1)
-		(exclude_from_sim yes)
-		(in_bom no)
+		(exclude_from_sim no)
+		(in_bom yes)
 		(on_board yes)
 		(dnp no)
@@
 		(at 359.41 195.58 180)
 		(unit 1)
-		(exclude_from_sim yes)
-		(in_bom no)
+		(exclude_from_sim no)
+		(in_bom yes)
 		(on_board yes)
 		(dnp no)
@@
 		(at 351.79 190.5 270)
 		(unit 1)
-		(exclude_from_sim yes)
-		(in_bom no)
+		(exclude_from_sim no)
+		(in_bom yes)
 		(on_board yes)
 		(dnp no)
@@
 			)
 		)
-		(property "Value" "White"
+		(property "Value" "Red"
 			(at 176.53 237.5534 90)
 			(effects
@@
 			)
 		)
-		(property "Manufacturer Product Number" "LTST-T180UWET"
+		(property "Manufacturer Product Number" "LTST-S270KRKT"
 			(at 173.99 236.22 90)
 			(effects
@@
 			)
 		)
-		(property "Part Number" "160-LTST-T180UWETCT-ND"
+		(property "Part Number" "160-1479-1-ND"
 			(at 173.99 236.22 90)
 			(effects
@@
 		(at 359.41 190.5 180)
 		(unit 1)
-		(exclude_from_sim yes)
-		(in_bom no)
+		(exclude_from_sim no)
+		(in_bom yes)
 		(on_board yes)
 		(dnp no)
@@
 			)
 		)
-		(property "Value" "Green"
+		(property "Value" "Yellow"
 			(at 370.332 171.958 0)
 			(effects
@@
 			)
 		)
-		(property "Manufacturer" "Kingbright"
+		(property "Manufacturer" "Lite-On Inc."
 			(at 359.41 172.72 0)
 			(effects
@@
 			)
 		)
-		(property "Manufacturer Product Number" "APT1608SGD3"
+		(property "Manufacturer Product Number" "LTST-C190KSKT"
 			(at 359.41 172.72 0)
 			(effects
@@
 			)
 		)
-		(property "Part Number" "754-APT1608SGD3CT-ND"
+		(property "Part Number" "160-1437-1-ND"
 			(at 359.41 172.72 0)
 			(effects
@@
 			)
 		)
-		(property "Value" "Green"
+		(property "Value" "White"
 			(at 369.824 166.116 0)
 			(effects
@@
 			)
 		)
-		(property "Manufacturer" "Kingbright"
+		(property "Manufacturer" "Lite-On Inc."
 			(at 359.41 167.64 0)
 			(effects
@@
 			)
 		)
-		(property "Manufacturer Product Number" "APT1608SGD3"
+		(property "Manufacturer Product Number" "LTST-T180UWET"
 			(at 359.41 167.64 0)
 			(effects
@@
 			)
 		)
-		(property "Part Number" "754-APT1608SGD3CT-ND"
+		(property "Part Number" "160-LTST-T180UWETCT-ND"
 			(at 359.41 167.64 0)
 			(effects
@@
 		(at 292.1 173.99 0)
 		(unit 1)
-		(exclude_from_sim no)
-		(in_bom yes)
+		(exclude_from_sim yes)
+		(in_bom no)
 		(on_board yes)
 		(dnp no)
@@
 			(at 292.1 173.99 0)
 			(effects
+				(font
+					(size 1.27 1.27)
+				)
+				(hide yes)
+			)
+		)
+		(property "Manufacturer" "Semtech Corporation"
+			(at 292.1 173.99 0)
+			(effects
+				(font
+					(size 1.27 1.27)
+				)
+				(hide yes)
+			)
+		)
+		(property "Manufacturer Product Number" "SRV05-4.TCT"
+			(at 292.1 173.99 0)
+			(effects
+				(font
+					(size 1.27 1.27)
+				)
+				(hide yes)
+			)
+		)
+		(property "DigiKey Part Number" "SRV05-4CT-ND"
+			(at 292.1 173.99 0)
+			(effects
